File: stm32-ble/stm32-ble.kicad_sch (KiCad schematic)
At the start: 49 parts, among them J1 USB_C_Receptacle_USB2.0, J2 TC2030, J3 Conn_01x04, J4 Conn_Coaxial, SW1 SW_Push, U1 USBLC6-2SC6, U2 MIC5365-3.3YD5, U3 STM32WB35CEU6A, X1 32khz768, X2 32MHz

Commit message: drc
Connections:
- net LSE_IN: now reaches C15.1, U3.2 (PC14), X1.2
- net LSE_OUT: now reaches C13.1, U3.3 (PC15), X1.1
Changed lines of the file:
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@@
+    (effects (font (size 0.5 0.5)) (justify left bottom))
+  )
+  (label "LSE_OUT" (at 165.1 133.35 0) (fields_autoplaced)
     (effects (font (size 0.5 0.5)) (justify left bottom))
   )
@@
     (effects (font (size 0.5 0.5)) (justify left bottom))
   )
+  (label "LSE_IN" (at 165.1 130.81 0) (fields_autoplaced)
+    (effects (font (size 0.5 0.5)) (justify left bottom))
+  )
